File: Ignix.kicad_sch (KiCad schematic)
At the start: 0 parts

Commit message: finished schem and pcb
Parts:
- added BT1: Battery_Cell, Battery:BatteryHolder_Keystone_3034_1x20mm, symbol Device:Battery_Cell
- added C1: 10µF, Capacitor_THT:CP_Radial_D8.0mm_P5.00mm, symbol Device:C
- added D1: LED, LED_THT:LED_D5.0mm, symbol Device:LED
- added M1: Motor_DC, Connector_PinHeader_2.54mm:PinHeader_1x02_P2.54mm_Vertical, symbol Motor:Motor_DC
- added Q1: NPN, Package_TO_SOT_THT:TO-92L_HandSolder, symbol Simulation_SPICE:NPN
- added Q2: PNP, Package_TO_SOT_THT:TO-92L_HandSolder, symbol Simulation_SPICE:PNP
- added R1, R3, R4: 4.7kΩ, Resistor_THT:R_Axial_DIN0207_L6.3mm_D2.5mm_P7.62mm_Horizontal, symbol Device:R
- added R2: 47kΩ, Resistor_THT:R_Axial_DIN0207_L6.3mm_D2.5mm_P7.62mm_Horizontal, symbol Device:R
- added R5: 220Ω, Resistor_THT:R_Axial_DIN0207_L6.3mm_D2.5mm_P7.62mm_Horizontal, symbol Device:R
- added RV1: 47kΩ, Potentiometer_THT:Potentiometer_Vishay_T73YP_Vertical, symbol Device:R_Potentiometer
- added SW1: SW_Push, Button_Switch_THT:SW_PUSH_6mm, symbol Switch:SW_Push
Connections:
- new net: Q1.2 (B), R2.1, RV1.1, RV1.2
- new net: R1.2, RV1.3
- new net: D1.2 (A), M1.1 (+), Q2.1 (C)
- new net: BT1.1 (+), C1.2, M1.2 (-), Q1.3 (E), R2.2, R5.2
- new net: C1.1, R1.1, SW1.2
- new net: Q1.1 (C), R3.2, R4.1
- new net: Q2.2 (B), R4.2
- new net: D1.1 (K), R5.1
- new net: BT1.2 (-), Q2.3 (E), R3.1, SW1.1
