File: Ignix.kicad_pcb (KiCad board)
At the start: 2 copper layers, 63.2 x 63.2 mm, 16 parts, among them M1 Motor_DC, Q1 NPN, Q2 PNP, SW1 SW_Push

Commit message: removed junk and updated FINAL pcb / schem
Parts:
- moved G*** 0.65 mm to (141.9, 68.5)
- moved G*** 0.57 mm to (108.8, 68.5)
